Commit message: feat: add camera but havent debug

File: mobile_robot/urdf/gazebo.xacro (robot description, xacro)
@@ -128,3 +128,72 @@
     </sensor>
   </gazebo>
+  <!-- ZED2 Stereo Camera -->
+  <!-- Camera trái -->
+  <gazebo reference="zed2_left_camera_optical_frame">
+    <sensor name="zed2_left_camera" type="camera">
+      <always_on>true</always_on>
+      <update_rate>30</update_rate>
+      <visualize>true</visualize>
+      <gz_frame_id>zed2_left_camera_optical_frame</gz_frame_id>
+      <!-- Topic -->
+      <topic>zed2/left/image_raw</topic>
+      <camera_info_topic>zed2/left/camera_info</camera_info_topic>
+      <camera>
+        <horizontal_fov>1.92</horizontal_fov>  <!-- ~110° -->
+        <vertical_fov>1.08</vertical_fov>      <!-- ~62° -->
+        <image>
+          <width>1280</width>
+          <height>720</height>
+          <format>R8G8B8</format>
+        </image>
+        <clip>
+          <near>0.05</near>
+          <far>50.0</far>
+        </clip>
+      </camera>
+      <!-- Noise -->
+      <noise>
+        <type>gaussian</type>
+        <mean>0.0</mean>
+        <stddev>0.003</stddev>
+      </noise>
+      <!-- Plugin camera Ignition -->
+      <plugin name="ignition::gazebo::systems::Camera"
+              filename="ignition-gazebo-camera-system"/>
+    </sensor>
+  </gazebo>
+  <!-- Camera phải -->
+  <gazebo reference="zed2_right_camera_optical_frame">
+    <sensor name="zed2_right_camera" type="camera">
+      <always_on>true</always_on>
+      <update_rate>30</update_rate>
+      <visualize>true</visualize>
+      <gz_frame_id>zed2_right_camera_optical_frame</gz_frame_id>
+      <!-- Topic -->
+      <topic>zed2/right/image_raw</topic>
+      <camera_info_topic>zed2/right/camera_info</camera_info_topic>
+      <camera>
+        <horizontal_fov>1.92</horizontal_fov>
+        <vertical_fov>1.08</vertical_fov>
+        <image>
+          <width>1280</width>
+          <height>720</height>
+          <format>R8G8B8</format>
+        </image>
+        <clip>
+          <near>0.05</near>
+          <far>50.0</far>
+        </clip>
+      </camera>
+      <!-- Noise -->
+      <noise>
+        <type>gaussian</type>
+        <mean>0.0</mean>
+        <stddev>0.003</stddev>
+      </noise>
+      <!-- Plugin camera Ignition -->
+      <plugin name="ignition::gazebo::systems::Camera"
+              filename="ignition-gazebo-camera-system"/>
+    </sensor>
+  </gazebo>
 </robot>

File: mobile_robot/urdf/new_robot_2.xacro (robot description, xacro)
@@ -340,3 +340,76 @@
     </joint>
     <!-- End IMU -->
+	<!--Zed2 Camera-->
+	<link name="zed2_link">
+	<visual>
+		<!-- Đẩy thân ZED2 ra trước 5cm để không trùng chassis -->
+		<origin xyz="0.05 0 0" rpy="0 0 0"/>
+		<geometry>
+		<box size="0.05 0.20 0.05"/>
+		</geometry>
+		<material name="red"/> <!-- đổi màu dễ nhìn -->
+	</visual>
+	<collision>
+		<origin xyz="0.05 0 0" rpy="0 0 0"/>
+		<geometry>
+		<box size="0.05 0.20 0.05"/>
+		</geometry>
+	</collision>
+	<inertial>
+		<mass value="0.25"/>
+		<origin xyz="0 0 0" rpy="0 0 0"/>
+		<inertia ixx="0.0001" iyy="0.0001" izz="0.0001"/>
+	</inertial>
+	</link>
+	<joint name="zed2_joint" type="fixed">
+		<parent link="base_link"/>
+		<child link="zed2_link"/>
+		<!-- Nhấc camera lên cao và ra trước robot -->
+		<origin xyz="0.20 0.0 0.40" rpy="0 0 0"/>
+	</joint>
+	<!-- Left Camera -->
+	<link name="zed2_left_camera_frame"/>
+	<joint name="zed2_left_camera_joint" type="fixed">
+		<parent link="zed2_link"/>
+		<child link="zed2_left_camera_frame"/>
+		<origin xyz="0 0.06 0" rpy="0 0 0"/>
+	</joint>
+	<link name="zed2_left_camera_optical_frame">
+		<visual>
+		<origin xyz="0 0 0" rpy="0 0 0"/>
+		<geometry>
+			<!-- Mắt trái -->
+			<cylinder radius="0.01" length="0.015"/>
+		</geometry>
+		<material name="black"/>
+		</visual>
+	</link>
+	<joint name="zed2_left_optical_joint" type="fixed">
+		<parent link="zed2_left_camera_frame"/>
+		<child link="zed2_left_camera_optical_frame"/>
+		<origin xyz="0 0 0" rpy="${-PI/2} 0 ${-PI/2}"/>
+	</joint>
+	<!-- Right Camera -->
+	<link name="zed2_right_camera_frame"/>
+	<joint name="zed2_right_camera_joint" type="fixed">
+		<parent link="zed2_link"/>
+		<child link="zed2_right_camera_frame"/>
+		<origin xyz="0 -0.06 0" rpy="0 0 0"/>
+	</joint>
+	<link name="zed2_right_camera_optical_frame">
+		<visual>
+		<origin xyz="0 0 0" rpy="0 0 0"/>
+		<geometry>
+			<!-- Mắt phải -->
+			<cylinder radius="0.01" length="0.015"/>
+		</geometry>
+		<material name="black"/>
+		</visual>
+	</link>
+	<joint name="zed2_right_optical_joint" type="fixed">
+		<parent link="zed2_right_camera_frame"/>
+		<child link="zed2_right_camera_optical_frame"/>
+		<origin xyz="0 0 0" rpy="${-PI/2} 0 ${-PI/2}"/>
+	</joint>
+	<!--  End ZED2 -->
 </robot>

Commit message: feat: have debugged camera and change link IMU on Camera

File: mobile_robot/urdf/gazebo.xacro (robot description, xacro)
@@ -129,71 +129,51 @@
   </gazebo>
   <!-- ZED2 Stereo Camera -->
-  <!-- Camera trái -->
-  <gazebo reference="zed2_left_camera_optical_frame">
-    <sensor name="zed2_left_camera" type="camera">
-      <always_on>true</always_on>
-      <update_rate>30</update_rate>
-      <visualize>true</visualize>
-      <gz_frame_id>zed2_left_camera_optical_frame</gz_frame_id>
-      <!-- Topic -->
-      <topic>zed2/left/image_raw</topic>
-      <camera_info_topic>zed2/left/camera_info</camera_info_topic>
-      <camera>
-        <horizontal_fov>1.92</horizontal_fov>  <!-- ~110° -->
-        <vertical_fov>1.08</vertical_fov>      <!-- ~62° -->
-        <image>
-          <width>1280</width>
-          <height>720</height>
-          <format>R8G8B8</format>
-        </image>
-        <clip>
-          <near>0.05</near>
-          <far>50.0</far>
-        </clip>
-      </camera>
-      <!-- Noise -->
-      <noise>
-        <type>gaussian</type>
-        <mean>0.0</mean>
-        <stddev>0.003</stddev>
-      </noise>
-      <!-- Plugin camera Ignition -->
-      <plugin name="ignition::gazebo::systems::Camera"
-              filename="ignition-gazebo-camera-system"/>
-    </sensor>
-  </gazebo>
-  <!-- Camera phải -->
-  <gazebo reference="zed2_right_camera_optical_frame">
-    <sensor name="zed2_right_camera" type="camera">
-      <always_on>true</always_on>
-      <update_rate>30</update_rate>
-      <visualize>true</visualize>
-      <gz_frame_id>zed2_right_camera_optical_frame</gz_frame_id>
-      <!-- Topic -->
-      <topic>zed2/right/image_raw</topic>
-      <camera_info_topic>zed2/right/camera_info</camera_info_topic>
-      <camera>
-        <horizontal_fov>1.92</horizontal_fov>
-        <vertical_fov>1.08</vertical_fov>
-        <image>
-          <width>1280</width>
-          <height>720</height>
-          <format>R8G8B8</format>
-        </image>
-        <clip>
-          <near>0.05</near>
-          <far>50.0</far>
-        </clip>
-      </camera>
-      <!-- Noise -->
-      <noise>
-        <type>gaussian</type>
-        <mean>0.0</mean>
-        <stddev>0.003</stddev>
-      </noise>
-      <!-- Plugin camera Ignition -->
-      <plugin name="ignition::gazebo::systems::Camera"
-              filename="ignition-gazebo-camera-system"/>
-    </sensor>
-  </gazebo>
+  <!-- Left camera -->
+<gazebo reference="zed2_left_camera_frame">
+  <sensor name="zed2_left_camera_sensor" type="camera">
+    <always_on>true</always_on>
+    <update_rate>30</update_rate>
+    <visualize>true</visualize>
+    <gz_frame_id>zed2_left_camera_frame</gz_frame_id>
+    <topic>zed2/left/image_raw</topic>
+    <camera_info_topic>zed2/left/camera_info</camera_info_topic>
+    <camera>
+      <horizontal_fov>1.92</horizontal_fov>
+      <vertical_fov>1.08</vertical_fov>
+      <image>
+        <width>1280</width>
+        <height>720</height>
+        <format>R8G8B8</format>
+      </image>
+      <clip><near>0.05</near><far>50.0</far></clip>
+    </camera>
+    <noise><type>gaussian</type><mean>0.0</mean><stddev>0.003</stddev></noise>
+    <plugin filename="ignition-gazebo-camera-system"
+            name="ignition::gazebo::systems::Camera"/>
+  </sensor>
+</gazebo>
+<!-- Right camera -->
+<gazebo reference="zed2_right_camera_frame">
+  <sensor name="zed2_right_camera_sensor" type="camera">
+    <always_on>true</always_on>
+    <update_rate>30</update_rate>
+    <visualize>true</visualize>
+    <gz_frame_id>zed2_right_camera_frame</gz_frame_id>
+    <topic>zed2/right/image_raw</topic>
+    <camera_info_topic>zed2/right/camera_info</camera_info_topic>
+    <camera>
+      <horizontal_fov>1.92</horizontal_fov>
+      <vertical_fov>1.08</vertical_fov>
+      <image>
+        <width>1280</width>
+        <height>720</height>
+        <format>R8G8B8</format>
+      </image>
+      <clip><near>0.05</near><far>50.0</far></clip>
+    </camera>
+    <noise><type>gaussian</type><mean>0.0</mean><stddev>0.003</stddev></noise>
+    <plugin filename="ignition-gazebo-camera-system"
+            name="ignition::gazebo::systems::Camera"/>
+  </sensor>
+</gazebo>
 </robot>

File: mobile_robot/urdf/new_robot_2.xacro (robot description, xacro)
@@ -332,84 +332,56 @@
         </visual>
     </link>
-	<!-- Imu -->
-    <link name="imu_link"/>
-    <joint name="imu_joint" type="fixed">
-        <parent link="base_link"/>
-        <child link="imu_link"/>
-        <origin xyz="0.0 0.0 0.0" rpy="0.0 0.0 0.0"/>
-    </joint>
-    <!-- End IMU -->
-	<!--Zed2 Camera-->
+	<!-- Thân ZED2 (body) -->
 	<link name="zed2_link">
-	<visual>
-		<!-- Đẩy thân ZED2 ra trước 5cm để không trùng chassis -->
-		<origin xyz="0.05 0 0" rpy="0 0 0"/>
-		<geometry>
-		<box size="0.05 0.20 0.05"/>
-		</geometry>
-		<material name="red"/> <!-- đổi màu dễ nhìn -->
-	</visual>
-	<collision>
-		<origin xyz="0.05 0 0" rpy="0 0 0"/>
-		<geometry>
-		<box size="0.05 0.20 0.05"/>
-		</geometry>
-	</collision>
-	<inertial>
-		<mass value="0.25"/>
-		<origin xyz="0 0 0" rpy="0 0 0"/>
-		<inertia ixx="0.0001" iyy="0.0001" izz="0.0001"/>
-	</inertial>
+		<visual>
+			<origin xyz="0 0 0" rpy="0 0 0"/>
+			<geometry>
+				<!-- 146.5 x 30 x 23 mm -->
+				<box size="0.03 0.1465 0.023"/>
+			</geometry>
+			<material name="grey"/>
+		</visual>
+		<collision>
+			<origin xyz="0 0 0" rpy="0 0 0"/>
+			<geometry>
+				<box size="0.03 0.1465 0.023"/>
+			</geometry>
+		</collision>
+		<inertial>
+			<mass value="0.5"/>
+			<origin xyz="0 0 0" rpy="0 0 0"/>
+			<inertia ixx="0.01" iyy="0.01" izz="0.01" ixy="0" ixz="0" iyz="0"/>
+		</inertial>
 	</link>
 	<joint name="zed2_joint" type="fixed">
 		<parent link="base_link"/>
 		<child link="zed2_link"/>
-		<!-- Nhấc camera lên cao và ra trước robot -->
-		<origin xyz="0.20 0.0 0.40" rpy="0 0 0"/>
+		<!-- đặt phía trước robot -->
+		<origin xyz="0.17 0.0 0.2"/>
 	</joint>
-	<!-- Left Camera -->
+	<!-- Left Camera (U26) -->
 	<link name="zed2_left_camera_frame"/>
 	<joint name="zed2_left_camera_joint" type="fixed">
 		<parent link="zed2_link"/>
 		<child link="zed2_left_camera_frame"/>
-		<origin xyz="0 0.06 0" rpy="0 0 0"/>
+		<!-- 9.3 mm từ mép trái: -0.07325 m so với tâm -->
+		<origin xyz="0 -0.07325 0"/>
 	</joint>
-	<link name="zed2_left_camera_optical_frame">
-		<visual>
-		<origin xyz="0 0 0" rpy="0 0 0"/>
-		<geometry>
-			<!-- Mắt trái -->
-			<cylinder radius="0.01" length="0.015"/>
-		</geometry>
-		<material name="black"/>
-		</visual>
-	</link>
-	<joint name="zed2_left_optical_joint" type="fixed">
-		<parent link="zed2_left_camera_frame"/>
-		<child link="zed2_left_camera_optical_frame"/>
-		<origin xyz="0 0 0" rpy="${-PI/2} 0 ${-PI/2}"/>
-	</joint>
-	<!-- Right Camera -->
+	<!-- Right Camera (U36) -->
 	<link name="zed2_right_camera_frame"/>
 	<joint name="zed2_right_camera_joint" type="fixed">
 		<parent link="zed2_link"/>
 		<child link="zed2_right_camera_frame"/>
-		<origin xyz="0 -0.06 0" rpy="0 0 0"/>
-	</joint>
-	<link name="zed2_right_camera_optical_frame">
-		<visual>
-		<origin xyz="0 0 0" rpy="0 0 0"/>
-		<geometry>
-			<!-- Mắt phải -->
-			<cylinder radius="0.01" length="0.015"/>
-		</geometry>
-		<material name="black"/>
-		</visual>
-	</link>
-	<joint name="zed2_right_optical_joint" type="fixed">
-		<parent link="zed2_right_camera_frame"/>
-		<child link="zed2_right_camera_optical_frame"/>
-		<origin xyz="0 0 0" rpy="${-PI/2} 0 ${-PI/2}"/>
+		<!-- 129.3 mm từ mép trái: +0.07325 m so với tâm -->
+		<origin xyz="0 0.07325 0"/>
 	</joint>
 	<!--  End ZED2 -->
+	<!-- Imu -->
+    <link name="imu_link"/>
+    <joint name="imu_joint" type="fixed">
+        <parent link="zed2_link"/>
+        <child link="imu_link"/>
+        <origin xyz="0 0.05 -0.0115" rpy="0 0 0"/>
+    </joint>
+    <!-- End IMU -->
 </robot>
