Commit message: feat: finish model but not yet zed and imu

File: mobile_robot/urdf/new_robot_3.xacro (robot description, xacro)
@@ -80,9 +80,9 @@
         <parent link="base_link"/>
         <child link="chassis"/>
-        <origin xyz="0.16 0.0 0.0"/>
+        <origin xyz="-0.16 0.0 0.0"/>
     </joint>
     <link name="chassis">
         <visual>
-            <origin xyz="-0.2055 0.0 0.07" rpy="0.0 0.0 0.0"/>
+            <origin xyz="0.2055 0.0 0.07" rpy="0.0 0.0 0.0"/>
             <geometry>
                  <box size="${body_length} ${body_width} ${body_height}"/>
@@ -91,5 +91,5 @@
         </visual>
         <collision>
-            <origin xyz="-0.2055 0.0 0.07" rpy="0.0 0.0 0.0"/>
+            <origin xyz="0.2055 0.0 0.07" rpy="0.0 0.0 0.0"/>
             <geometry>
                  <box size="${body_length} ${body_width} ${body_height}"/>
@@ -97,5 +97,5 @@
         </collision>
         <inertial>
-            <origin xyz="-0.2055 0.0 0.07" rpy="0.0 0.0 0.0"/>
+            <origin xyz="0.2055 0.0 0.07" rpy="0.0 0.0 0.0"/>
             <mass value="${body_mass}"/>
             <xacro:box_inertia m="${body_mass}" l="${body_length}" w="${body_width}" h="${body_height}"/>
@@ -106,5 +106,5 @@
         <parent link="base_link"/>
         <child link="right_wheel"/>
-        <origin xyz="0.03 -0.23 0.0" rpy="${PI/2} 0 0"/>
+        <origin xyz="-0.03 -0.23 0.0" rpy="${PI/2} 0 0"/>
         <axis xyz="0 0 -1"/>
     </joint>
@@ -130,5 +130,5 @@
        	<parent link="base_link"/>
         <child link="left_wheel"/>
-        <origin xyz="0.03 0.23 0.0" rpy="${-PI/2} 0.0 0.0"/>
+        <origin xyz="-0.03 0.23 0.0" rpy="${-PI/2} 0.0 0.0"/>
         <axis xyz="0 0 1"/>
     </joint>
@@ -155,5 +155,5 @@
          	<parent link="base_link"/>
          	<child link="above_base_caster"/>
-         	<origin xyz="-0.025 0.0 0.40" rpy="0 0 0"/>
+         	<origin xyz="0.025 0.0 0.40" rpy="0 0 0"/>
     </joint>
 	<link name = "above_base_caster" >
@@ -180,5 +180,5 @@
         <parent link="base_link"/>
         <child link="right_base_caster"/>
-        <origin xyz="-0.025 0.19 0.22" rpy="0 0 0"/>
+        <origin xyz="0.025 0.19 0.22" rpy="0 0 0"/>
     </joint>
 	<link name = "right_base_caster" >
@@ -205,5 +205,5 @@
         <parent link="base_link"/>
         <child link="left_base_caster"/>
-        <origin xyz="-0.025 -0.19 0.22" rpy="0 0 0"/>
+        <origin xyz="0.025 -0.19 0.22" rpy="0 0 0"/>
     </joint>
 	<link name = "left_base_caster" >
@@ -230,5 +230,5 @@
         <parent link="base_link"/>
         <child link="back_base_caster"/>
-        <origin xyz="0.1 0 0.22" rpy="0 0 0"/>
+        <origin xyz="-0.1 0 0.22" rpy="0 0 0"/>
     </joint>
 	<link name = "back_base_caster" >
@@ -278,5 +278,6 @@
 <!--lidar-->
     <joint name="joint_scan" type="fixed">
-        <origin xyz="0 0.0 ${body_height +0.25+ 0.009}" rpy="0.0 0.0 0.0"/>
+        <origin xyz="0 0.0 ${body_height +0.25+ 0.009}" rpy="0.0 0.0 3.14159"/>     <!--0.215 = 0.2 + 0.03/2-->
+        <!-- <origin xyz="0 0.0 ${body_height +0.25+ 0.009}" rpy="0.0 0.0 -0.3837777777777778"/> -->
         <parent link="base_link"/>
         <child link="laser"/>
@@ -306,5 +307,5 @@
         <parent link="chassis"/>
         <child link="face_link"/>
-        <origin xyz="${-body_length} 0 ${body_height/2}" rpy="0 0 0"/>
+        <origin xyz="-${body_length} 0 ${body_height/2}" rpy="0 0 0"/>
     </joint>
     <link name="face_link">
@@ -356,6 +357,6 @@
 		<parent link="base_link"/>
 		<child link="zed2_link"/>
-		<!-- đặt phía trước robot, gần 2 bánh vi sai -->
-		<origin xyz="0.08 0.0 0.2"/>
+		<!-- đặt phía trước robot -->
+		<origin xyz="0.17 0.0 0.2"/>
 	</joint>
 	<!-- Left Camera (U26) -->
