Commit message: feat: add funsion not finish

File: mobile_robot/urdf/new_robot_2.xacro (robot description, xacro)
@@ -356,6 +356,6 @@
 		<parent link="base_link"/>
 		<child link="zed2_link"/>
-		<!-- đặt phía trước robot, gần 2 bánh vi sai -->
-		<origin xyz="0.08 0.0 0.2"/>
+		<!-- Camera dời ra phía trước và cao hơn để nhìn thấy ArUco markers -->
+		<origin xyz="0.10 0.0 0.35"/>
 	</joint>
 	<!-- Left Camera (U26) -->

Commit message: Add pkg agv_zed2

File: mobile_robot/urdf/new_robot_2.xacro (robot description, xacro)
@@ -357,5 +357,5 @@
 		<child link="zed2_link"/>
 		<!-- đặt phía trước robot, gần 2 bánh vi sai -->
-		<origin xyz="0.08 0.0 0.2"/>
+		<origin xyz="0.1 0.0 0.2"/>
 	</joint>
 	<!-- Left Camera (U26) -->

Commit message: feat: fix lidar scan wrong

File: mobile_robot/urdf/new_robot_2.xacro (robot description, xacro)
@@ -277,9 +277,9 @@
 	</link>
 <!--lidar-->
-    <joint name="joint_scan" type="fixed">
-        <origin xyz="0 0.0 ${body_height +0.25+ 0.009}" rpy="0.0 0.0 0.0"/>
-        <parent link="base_link"/>
-        <child link="laser"/>
-    </joint>
+	<joint name="joint_scan" type="fixed">
+		<origin xyz="0 0.0 ${body_height +0.25+ 0.009}" rpy="0.0 0.0 ${PI}"/>
+		<parent link="base_link"/>
+		<child link="laser"/>
+	</joint>
     <link name="laser">
         <visual>

Commit message: feat: fix scan lidar wrong

File: mobile_robot/urdf/new_robot_2.xacro (robot description, xacro)
@@ -278,5 +278,5 @@
 <!--lidar-->
 	<joint name="joint_scan" type="fixed">
-		<origin xyz="0 0.0 ${body_height +0.25+ 0.009}" rpy="0.0 0.0 ${PI}"/>
+		<origin xyz="0 0 0" rpy="0 0 ${PI}"/>
 		<parent link="base_link"/>
 		<child link="laser"/>

Commit message: feat: update scan

File: mobile_robot/urdf/new_robot_2.xacro (robot description, xacro)
@@ -278,5 +278,5 @@
 <!--lidar-->
 	<joint name="joint_scan" type="fixed">
-		<origin xyz="0 0 0" rpy="0 0 ${PI}"/>
+		<origin xyz="0 0 0" rpy="0 0 0"/>
 		<parent link="base_link"/>
 		<child link="laser"/>

Commit message: update scan part n

File: mobile_robot/urdf/new_robot_2.xacro (robot description, xacro)
@@ -278,5 +278,5 @@
 <!--lidar-->
 	<joint name="joint_scan" type="fixed">
-		<origin xyz="0 0 0" rpy="0 0 0"/>
+		<origin xyz="0 0 0" rpy="0 0 ${PI}"/>
 		<parent link="base_link"/>
 		<child link="laser"/>

Commit message: feat: fix urdf

File: mobile_robot/urdf/new_robot_2.xacro (robot description, xacro)
@@ -36,6 +36,6 @@
 	</material>
 <!--define physical properties for robot-->
-	<xacro:property name="body_length" value="0.31"/>
-	<xacro:property name="body_width" value="0.4"/>
+	<xacro:property name="body_length" value="0.38"/>
+	<xacro:property name="body_width" value="0.26"/>
 	<xacro:property name="body_height" value="0.2"/>
 	<xacro:property name="body_mass" value="12"/>
@@ -44,8 +44,8 @@
 	<xacro:property name="base_caster_height" value="0.37"/>
 	<xacro:property name="above_base_caster_length" value="0.25"/>
-	<xacro:property name="above_base_caster_width" value="0.4"/>
+	<xacro:property name="above_base_caster_width" value="0.26"/>
 	<xacro:property name="above_base_caster_height" value="0.0075"/>
 	<xacro:property name="back_base_caster_length" value="0.0075"/>
-	<xacro:property name="back_base_caster_width" value="0.4"/>
+	<xacro:property name="back_base_caster_width" value="0.26"/>
 	<xacro:property name="back_base_caster_height" value="0.37"/>
 	<xacro:property name="wheel_radius" value="0.05"/>

Commit message: feat: urdf fix done

File: mobile_robot/urdf/new_robot_2.xacro (robot description, xacro)
@@ -36,6 +36,6 @@
 	</material>
 <!--define physical properties for robot-->
-	<xacro:property name="body_length" value="0.38"/>
-	<xacro:property name="body_width" value="0.26"/>
+	<xacro:property name="body_length" value="0.33"/>
+	<xacro:property name="body_width" value="0.38"/>
 	<xacro:property name="body_height" value="0.2"/>
 	<xacro:property name="body_mass" value="12"/>
@@ -44,13 +44,13 @@
 	<xacro:property name="base_caster_height" value="0.37"/>
 	<xacro:property name="above_base_caster_length" value="0.25"/>
-	<xacro:property name="above_base_caster_width" value="0.26"/>
+	<xacro:property name="above_base_caster_width" value="0.38"/>
 	<xacro:property name="above_base_caster_height" value="0.0075"/>
 	<xacro:property name="back_base_caster_length" value="0.0075"/>
-	<xacro:property name="back_base_caster_width" value="0.26"/>
+	<xacro:property name="back_base_caster_width" value="0.38"/>
 	<xacro:property name="back_base_caster_height" value="0.37"/>
 	<xacro:property name="wheel_radius" value="0.05"/>
 	<xacro:property name="wheel_width" value="0.03"/>
 	<xacro:property name="wheel_mass" value="0.3"/>
-	<xacro:property name="wheel_separation" value="0.46"/>
+	<xacro:property name="wheel_separation" value="0.42"/>
 	<xacro:property name="PI" value="3.1415926535897931"/>
 	<xacro:macro name="cylinder_inertia" params="m r h">
@@ -106,5 +106,5 @@
         <parent link="base_link"/>
         <child link="right_wheel"/>
-        <origin xyz="0.03 -0.23 0.0" rpy="${PI/2} 0 0"/>
+        <origin xyz="0.03 -0.21 0.0" rpy="${PI/2} 0 0"/>
         <axis xyz="0 0 -1"/>
     </joint>
@@ -130,5 +130,5 @@
        	<parent link="base_link"/>
         <child link="left_wheel"/>
-        <origin xyz="0.03 0.23 0.0" rpy="${-PI/2} 0.0 0.0"/>
+        <origin xyz="0.03 0.21 0.0" rpy="${-PI/2} 0.0 0.0"/>
         <axis xyz="0 0 1"/>
     </joint>
@@ -150,105 +150,6 @@
         </inertial>
 	</link>
-<!--base caster-->
-	<!--above-->
-	<joint name="above_base_caster_joint" type="fixed">
-         	<parent link="base_link"/>
-         	<child link="above_base_caster"/>
-         	<origin xyz="-0.025 0.0 0.40" rpy="0 0 0"/>
-    </joint>
-	<link name = "above_base_caster" >
-		<visual>
-			<geometry>
-				<box size="${above_base_caster_length} ${above_base_caster_width} ${above_base_caster_height}"/>
-			</geometry>
-			<material name = "orange" />
-		</visual>
-		<collision>
-			<geometry>
-				<box size="${above_base_caster_length} ${above_base_caster_width} ${above_base_caster_height}"/>
-			</geometry>
-		</collision>
-		<inertial>
-            <mass value="0.2" />
-            <inertia ixx="0.1" ixy="0.0" ixz="0.0"
-                iyy="0.1" iyz="0.0"
-                izz="0.1" />
-        	</inertial>
-	</link>
+<!--base caster - REMOVED orange panels-->
 	<!--right-->
-	<joint name="right_base_caster_joint" type="fixed">
-        <parent link="base_link"/>
-        <child link="right_base_caster"/>
-        <origin xyz="-0.025 0.19 0.22" rpy="0 0 0"/>
-    </joint>
-	<link name = "right_base_caster" >
-		<visual>
-			<geometry>
-				<box size="${base_caster_length} ${base_caster_width} ${base_caster_height}"/>
-			</geometry>
-			<material name = "orange" />
-		</visual>
-		<collision>
-			<geometry>
-				<box size="${base_caster_length} ${base_caster_width} ${base_caster_height}"/>
-			</geometry>
-		</collision>
-		<inertial>
-        	<mass value="0.2" />
-            <inertia ixx="0.1" ixy="0.0" ixz="0.0"
-                iyy="0.1" iyz="0.0"
-                izz="0.1" />
-        	</inertial>
-	</link>
-	<!--left-->
-	<joint name="left_base_caster_joint" type="fixed">
-        <parent link="base_link"/>
-        <child link="left_base_caster"/>
-        <origin xyz="-0.025 -0.19 0.22" rpy="0 0 0"/>
-    </joint>
-	<link name = "left_base_caster" >
-		<visual>
-			<geometry>
-				<box size="${base_caster_length} ${base_caster_width} ${base_caster_height}"/>
-			</geometry>
-			<material name = "orange" />
-		</visual>
-		<collision>
-			<geometry>
-				<box size="${base_caster_length} ${base_caster_width} ${base_caster_height}"/>
-			</geometry>
-		</collision>
-		<inertial>
-            <mass value="0.2" />
-            <inertia ixx="0.1" ixy="0.0" ixz="0.0"
-                iyy="0.1" iyz="0.0"
-                izz="0.1" />
-        </inertial>
-	</link>
-	<!--back-->
-	<joint name="back_base_caster_joint" type="fixed">
-        <parent link="base_link"/>
-        <child link="back_base_caster"/>
-        <origin xyz="0.1 0 0.22" rpy="0 0 0"/>
-    </joint>
-	<link name = "back_base_caster" >
-		<visual>
-			<geometry>
-				<box size="${back_base_caster_length} ${back_base_caster_width} ${back_base_caster_height}"/>
-			</geometry>
-			<material name = "orange" />
-		</visual>
-		<collision>
-			<geometry>
-				<box size="${base_caster_length} ${base_caster_width} ${base_caster_height}"/>
-			</geometry>
-		</collision>
-		<inertial>
-            <mass value="0.5" />
-            <inertia ixx="0.1" ixy="0.0" ixz="0.0"
-            	iyy="0.1" iyz="0.0"
-                izz="0.1" />
-        	</inertial>
-	</link>
 <!--caster wheel-->
 	<joint name = "caster_wheel_joint" type = "fixed" >
@@ -278,5 +179,5 @@
 <!--lidar-->
 	<joint name="joint_scan" type="fixed">
-		<origin xyz="0 0 0" rpy="0 0 ${PI}"/>
+		<origin xyz="0 0 0.26" rpy="0 0 ${PI}"/>
 		<parent link="base_link"/>
 		<child link="laser"/>
@@ -356,6 +257,6 @@
 		<parent link="base_link"/>
 		<child link="zed2_link"/>
-		<!-- Camera dời ra phía trước và cao hơn để nhìn thấy ArUco markers -->
-		<origin xyz="0.10 0.0 0.35"/>
+		<!-- Camera 3cm above body top (body top at 0.17) -->
+		<origin xyz="0.10 0.0 0.20"/>
 	</joint>
 	<!-- Left Camera (U26) -->

Commit message: feat: final urdf

File: mobile_robot/urdf/new_robot_2.xacro (robot description, xacro)
@@ -40,13 +40,4 @@
 	<xacro:property name="body_height" value="0.2"/>
 	<xacro:property name="body_mass" value="12"/>
-	<xacro:property name="base_caster_length" value="0.25"/>
-	<xacro:property name="base_caster_width" value="0.01"/>
-	<xacro:property name="base_caster_height" value="0.37"/>
-	<xacro:property name="above_base_caster_length" value="0.25"/>
-	<xacro:property name="above_base_caster_width" value="0.38"/>
-	<xacro:property name="above_base_caster_height" value="0.0075"/>
-	<xacro:property name="back_base_caster_length" value="0.0075"/>
-	<xacro:property name="back_base_caster_width" value="0.38"/>
-	<xacro:property name="back_base_caster_height" value="0.37"/>
 	<xacro:property name="wheel_radius" value="0.05"/>
 	<xacro:property name="wheel_width" value="0.03"/>
@@ -150,6 +141,4 @@
         </inertial>
 	</link>
-<!--base caster - REMOVED orange panels-->
-	<!--right-->
 <!--caster wheel-->
 	<joint name = "caster_wheel_joint" type = "fixed" >
@@ -202,33 +191,4 @@
             <inertia ixx="0.01" ixy="0.0" ixz="0.0" iyy="0.01" iyz="0.0" izz="0.01"/>
         </inertial>
-    </link>
-<!--face robot-->
-    <joint name="face_joint" type="fixed">
-        <parent link="chassis"/>
-        <child link="face_link"/>
-        <origin xyz="${-body_length} 0 ${body_height/2}" rpy="0 0 0"/>
-    </joint>
-    <link name="face_link">
-        <visual>
-            <origin xyz="0.05 0.07 -0.075" rpy="0 ${PI/2} 0"/>
-            <geometry>
-                <cylinder radius="0.025" length="0.002"/>
-            </geometry>
-            <material name="white"/>
-        </visual>
-        <visual>
-            <origin xyz="0.05 -0.07 -0.075" rpy="0 ${PI/2} 0"/>
-            <geometry>
-                <cylinder radius="0.025" length="0.002"/>
-            </geometry>
-            <material name="white"/>
-        </visual>
-        <visual>
-            <origin xyz="0.05 0.0 0.0" rpy="0 ${1.5} 0"/>
-            <geometry>
-                <cylinder radius="0.03" length="0.02"/>
-            </geometry>
-            <material name="red"/>
-        </visual>
     </link>
 	<!-- Thân ZED2 (body) -->

Commit message: fix change orientation lidar

File: mobile_robot/urdf/new_robot_2.xacro (robot description, xacro)
@@ -278,5 +278,5 @@
 <!--lidar-->
     <joint name="joint_scan" type="fixed">
-        <origin xyz="0 0.0 ${body_height +0.25+ 0.009}" rpy="0.0 0.0 0.0"/>
+        <origin xyz="0 0.0 ${body_height +0.25+ 0.009}" rpy="0.0 0.0 ${PI}"/>
         <parent link="base_link"/>
         <child link="laser"/>

Commit message: feat: change imu_link

File: mobile_robot/urdf/new_robot_2.xacro (robot description, xacro)
@@ -237,10 +237,10 @@
 	</joint>
 	<!--  End ZED2 -->
-	<!-- Imu -->
+	<!-- IMU (trên mặt robot, phía trước base_link) -->
     <link name="imu_link"/>
     <joint name="imu_joint" type="fixed">
-        <parent link="zed2_link"/>
+        <parent link="base_link"/>
         <child link="imu_link"/>
-        <origin xyz="0 0.05 -0.0115" rpy="0 0 0"/>
+        <origin xyz="0.13 0.0 0.27" rpy="0 0 0"/>
     </joint>
     <!-- End IMU -->
