Commit message: feat: update urdf ver1

File: mobile_robot/urdf/new_robot_2.xacro (robot description, xacro)
@@ -36,8 +36,15 @@
 	</material>
 <!--define physical properties for robot-->
-	<xacro:property name="body_length" value="0.33"/>
-	<xacro:property name="body_width" value="0.38"/>
-	<xacro:property name="body_height" value="0.2"/>
-	<xacro:property name="body_mass" value="12"/>
+	<xacro:property name="body_length" value="0.3"/>
+	<xacro:property name="body_width" value="0.4"/>
+	<xacro:property name="body_height" value="0.3"/>
+	<xacro:property name="body_mass" value="15"/>
+	<!-- Frame structure properties (20x20cm grid) -->
+	<xacro:property name="frame_beam_radius" value="0.008"/>
+	<xacro:property name="frame_beam_mass" value="0.2"/>
+	<xacro:property name="frame_beam_20" value="0.02"/>
+	<xacro:property name="frame_beam_40" value="0.04"/>
+	<xacro:property name="mica_sheet_thickness" value="0.005"/>
+	<xacro:property name="mica_mass" value="0.2"/>
 	<xacro:property name="wheel_radius" value="0.05"/>
 	<xacro:property name="wheel_width" value="0.03"/>
@@ -67,28 +74,187 @@
        	<origin xyz="0.0 0.0 0.0"/>
     </link>
-<!--chassis link-->
+<!--chassis link - Frame Structure with Grid-->
     <joint name="chassis_joint" type="fixed">
         <parent link="base_link"/>
         <child link="chassis"/>
-        <origin xyz="0.16 0.0 0.0"/>
+        <origin xyz="0.0 0.0 0.0"/>
     </joint>
     <link name="chassis">
         <visual>
-            <origin xyz="-0.2055 0.0 0.07" rpy="0.0 0.0 0.0"/>
-            <geometry>
-                 <box size="${body_length} ${body_width} ${body_height}"/>
-            </geometry>
-            <material name="yellow"/>
-        </visual>
-        <collision>
-            <origin xyz="-0.2055 0.0 0.07" rpy="0.0 0.0 0.0"/>
-            <geometry>
-                 <box size="${body_length} ${body_width} ${body_height}"/>
-            </geometry>
-        </collision>
-        <inertial>
-            <origin xyz="-0.2055 0.0 0.07" rpy="0.0 0.0 0.0"/>
-            <mass value="${body_mass}"/>
-            <xacro:box_inertia m="${body_mass}" l="${body_length}" w="${body_width}" h="${body_height}"/>
+            <origin xyz="0.0 0.0 0.0" rpy="0.0 0.0 0.0"/>
+            <geometry>
+                 <box size="${body_length} ${body_width} ${mica_sheet_thickness}"/>
+            </geometry>
+            <material name="white"/>
+        </visual>
+        <collision>
+            <origin xyz="0.0 0.0 0.0" rpy="0.0 0.0 0.0"/>
+            <geometry>
+                 <box size="${body_length} ${body_width} ${mica_sheet_thickness}"/>
+            </geometry>
+        </collision>
+        <inertial>
+            <origin xyz="0.0 0.0 0.0" rpy="0.0 0.0 0.0"/>
+            <mass value="${mica_mass}"/>
+            <xacro:box_inertia m="${mica_mass}" l="${body_length}" w="${body_width}" h="${mica_sheet_thickness}"/>
+        </inertial>
+    </link>
+    <!-- Vertical support posts (corners) -->
+    <!-- Front Left Post -->
+    <joint name="post_fl_joint" type="fixed">
+        <parent link="base_link"/>
+        <child link="post_fl"/>
+        <origin xyz="0.15 -0.2 0.15"/>
+    </joint>
+    <link name="post_fl">
+        <visual>
+            <origin xyz="0.0 0.0 0.0" rpy="0.0 0.0 0.0"/>
+            <geometry>
+                <box size="${frame_beam_20} ${frame_beam_20} ${body_height}"/>
+            </geometry>
+            <material name="aluminium"/>
+        </visual>
+        <collision>
+            <origin xyz="0.0 0.0 0.0" rpy="0.0 0.0 0.0"/>
+            <geometry>
+                <box size="${frame_beam_20} ${frame_beam_20} ${body_height}"/>
+            </geometry>
+        </collision>
+        <inertial>
+            <origin xyz="0.0 0.0 0.0" rpy="0.0 0.0 0.0"/>
+            <mass value="${frame_beam_mass}"/>
+            <xacro:box_inertia m="${frame_beam_mass}" l="${frame_beam_20}" w="${frame_beam_20}" h="${body_height}"/>
+        </inertial>
+    </link>
+    <!-- Front Right Post -->
+    <joint name="post_fr_joint" type="fixed">
+        <parent link="base_link"/>
+        <child link="post_fr"/>
+        <origin xyz="0.15 0.2 0.15"/>
+    </joint>
+    <link name="post_fr">
+        <visual>
+            <origin xyz="0.0 0.0 0.0" rpy="0.0 0.0 0.0"/>
+            <geometry>
+                <box size="${frame_beam_20} ${frame_beam_20} ${body_height}"/>
+            </geometry>
+            <material name="aluminium"/>
+        </visual>
+        <collision>
+            <origin xyz="0.0 0.0 0.0" rpy="0.0 0.0 0.0"/>
+            <geometry>
+                <box size="${frame_beam_20} ${frame_beam_20} ${body_height}"/>
+            </geometry>
+        </collision>
+        <inertial>
+            <origin xyz="0.0 0.0 0.0" rpy="0.0 0.0 0.0"/>
+            <mass value="${frame_beam_mass}"/>
+            <xacro:box_inertia m="${frame_beam_mass}" l="${frame_beam_20}" w="${frame_beam_20}" h="${body_height}"/>
+        </inertial>
+    </link>
+    <!-- Back Left Post -->
+    <joint name="post_bl_joint" type="fixed">
+        <parent link="base_link"/>
+        <child link="post_bl"/>
+        <origin xyz="-0.15 -0.2 0.15"/>
+    </joint>
+    <link name="post_bl">
+        <visual>
+            <origin xyz="0.0 0.0 0.0" rpy="0.0 0.0 0.0"/>
+            <geometry>
+                <box size="${frame_beam_20} ${frame_beam_20} ${body_height}"/>
+            </geometry>
+            <material name="aluminium"/>
+        </visual>
+        <collision>
+            <origin xyz="0.0 0.0 0.0" rpy="0.0 0.0 0.0"/>
+            <geometry>
+                <box size="${frame_beam_20} ${frame_beam_20} ${body_height}"/>
+            </geometry>
+        </collision>
+        <inertial>
+            <origin xyz="0.0 0.0 0.0" rpy="0.0 0.0 0.0"/>
+            <mass value="${frame_beam_mass}"/>
+            <xacro:box_inertia m="${frame_beam_mass}" l="${frame_beam_20}" w="${frame_beam_20}" h="${body_height}"/>
+        </inertial>
+    </link>
+    <!-- Back Right Post -->
+    <joint name="post_br_joint" type="fixed">
+        <parent link="base_link"/>
+        <child link="post_br"/>
+        <origin xyz="-0.15 0.2 0.15"/>
+    </joint>
+    <link name="post_br">
+        <visual>
+            <origin xyz="0.0 0.0 0.0" rpy="0.0 0.0 0.0"/>
+            <geometry>
+                <box size="${frame_beam_20} ${frame_beam_20} ${body_height}"/>
+            </geometry>
+            <material name="aluminium"/>
+        </visual>
+        <collision>
+            <origin xyz="0.0 0.0 0.0" rpy="0.0 0.0 0.0"/>
+            <geometry>
+                <box size="${frame_beam_20} ${frame_beam_20} ${body_height}"/>
+            </geometry>
+        </collision>
+        <inertial>
+            <origin xyz="0.0 0.0 0.0" rpy="0.0 0.0 0.0"/>
+            <mass value="${frame_beam_mass}"/>
+            <xacro:box_inertia m="${frame_beam_mass}" l="${frame_beam_20}" w="${frame_beam_20}" h="${body_height}"/>
+        </inertial>
+    </link>
+    <!-- Middle vertical posts (20x20cm grid) -->
+    <!-- Mica layers at different heights -->
+    <!-- Middle Layer -->
+    <joint name="layer_middle_joint" type="fixed">
+        <parent link="base_link"/>
+        <child link="layer_middle"/>
+        <origin xyz="0.0 0.0 0.15" rpy="0.0 0.0 0.0"/>
+    </joint>
+    <link name="layer_middle">
+        <visual>
+            <origin xyz="0.0 0.0 0.0" rpy="0.0 0.0 0.0"/>
+            <geometry>
+                 <box size="${body_length} ${body_width} ${mica_sheet_thickness}"/>
+            </geometry>
+            <material name="white"/>
+        </visual>
+        <collision>
+            <origin xyz="0.0 0.0 0.0" rpy="0.0 0.0 0.0"/>
+            <geometry>
+                 <box size="${body_length} ${body_width} ${mica_sheet_thickness}"/>
+            </geometry>
+        </collision>
+        <inertial>
+            <origin xyz="0.0 0.0 0.0" rpy="0.0 0.0 0.0"/>
+            <mass value="${mica_mass}"/>
+            <xacro:box_inertia m="${mica_mass}" l="${body_length}" w="${body_width}" h="${mica_sheet_thickness}"/>
+        </inertial>
+    </link>
+    <!-- Top Layer -->
+    <joint name="layer_top_joint" type="fixed">
+        <parent link="base_link"/>
+        <child link="layer_top"/>
+        <origin xyz="0.0 0.0 0.295" rpy="0.0 0.0 0.0"/>
+    </joint>
+    <link name="layer_top">
+        <visual>
+            <origin xyz="0.0 0.0 0.0" rpy="0.0 0.0 0.0"/>
+            <geometry>
+                 <box size="${body_length} ${body_width} ${mica_sheet_thickness}"/>
+            </geometry>
+            <material name="white"/>
+        </visual>
+        <collision>
+            <origin xyz="0.0 0.0 0.0" rpy="0.0 0.0 0.0"/>
+            <geometry>
+                 <box size="${body_length} ${body_width} ${mica_sheet_thickness}"/>
+            </geometry>
+        </collision>
+        <inertial>
+            <origin xyz="0.0 0.0 0.0" rpy="0.0 0.0 0.0"/>
+            <mass value="${mica_mass}"/>
+            <xacro:box_inertia m="${mica_mass}" l="${body_length}" w="${body_width}" h="${mica_sheet_thickness}"/>
         </inertial>
     </link>
@@ -97,5 +263,5 @@
         <parent link="base_link"/>
         <child link="right_wheel"/>
-        <origin xyz="0.03 -0.21 0.0" rpy="${PI/2} 0 0"/>
+        <origin xyz="0.1 -0.23 -0.02" rpy="${PI/2} 0 0"/>
         <axis xyz="0 0 -1"/>
     </joint>
@@ -121,5 +287,5 @@
        	<parent link="base_link"/>
         <child link="left_wheel"/>
-        <origin xyz="0.03 0.21 0.0" rpy="${-PI/2} 0.0 0.0"/>
+        <origin xyz="0.1 0.23 -0.02" rpy="${-PI/2} 0.0 0.0"/>
         <axis xyz="0 0 1"/>
     </joint>
@@ -141,32 +307,30 @@
         </inertial>
 	</link>
-<!--caster wheel-->
-	<joint name = "caster_wheel_joint" type = "fixed" >
-		<parent link = "base_link" />
-		<child link = "caster_wheel" />
-		<origin xyz = "-0.13 0 0.0" />
+<!--caster wheel - free castor at back-->
+	<joint name="caster_wheel_joint" type="fixed">
+		<parent link="base_link"/>
+		<child link="caster_wheel"/>
+		<origin xyz="-0.1 0.0 -0.035"/>
 	</joint>
-	<link name = "caster_wheel" >
+	<link name="caster_wheel">
 		<visual>
 			<geometry>
-				<sphere radius = "0.05" />
+				<sphere radius="0.035"/>
 			</geometry>
-			<material name = "red" />
+			<material name="red"/>
 		</visual>
 		<collision>
 			<geometry>
-				<sphere radius = "0.05" />
+				<sphere radius="0.035"/>
 			</geometry>
 		</collision>
 		<inertial>
-            <mass value="0.1" />
-            <inertia ixx="0.1" ixy="0.0" ixz="0.0"
-                iyy="0.1" iyz="0.0"
-                izz="0.1" />
-        </inertial>
+			<mass value="0.08"/>
+			<inertia ixx="0.0001" ixy="0.0" ixz="0.0" iyy="0.0001" iyz="0.0" izz="0.0001"/>
+		</inertial>
 	</link>
 <!--lidar-->
 	<joint name="joint_scan" type="fixed">
-		<origin xyz="0 0 0.26" rpy="0 0 ${PI}"/>
+		<origin xyz="0.0 0.0 0.4" rpy="0 0 0"/>
 		<parent link="base_link"/>
 		<child link="laser"/>
@@ -174,5 +338,5 @@
     <link name="laser">
         <visual>
-            <origin xyz="0.01 0.0 -0.04" rpy="0.0 0.0 0.0"/>
+            <origin xyz="0.0 0.0 0.0" rpy="0.0 0.0 0.0"/>
             <geometry>
                 <cylinder radius="0.04" length="0.03"/>
@@ -181,5 +345,5 @@
         </visual>
         <collision>
-            <origin xyz="0.01 0.0 -0.04" rpy="0.0 0.0 0.0"/>
+            <origin xyz="0.0 0.0 0.0" rpy="0.0 0.0 0.0"/>
             <geometry>
                 <cylinder radius="0.04" length="0.03"/>
@@ -187,5 +351,5 @@
         </collision>
         <inertial>
-            <origin xyz="0.01 0.0 -0.04" rpy="0.0 0.0 0.0"/>
+            <origin xyz="0.0 0.0 0.0" rpy="0.0 0.0 0.0"/>
             <mass value="0.114"/>
             <inertia ixx="0.01" ixy="0.0" ixz="0.0" iyy="0.01" iyz="0.0" izz="0.01"/>
@@ -217,6 +381,6 @@
 		<parent link="base_link"/>
 		<child link="zed2_link"/>
-		<!-- Camera 3cm above body top (body top at 0.17) -->
-		<origin xyz="0.10 0.0 0.20"/>
+		<!-- Camera at 15cm from center forward on robot -->
+		<origin xyz="0.15 0.0 0.35"/>
 	</joint>
 	<!-- Left Camera (U26) -->
@@ -237,10 +401,10 @@
 	</joint>
 	<!--  End ZED2 -->
-	<!-- IMU (trên mặt robot, phía trước base_link) -->
+	<!-- IMU (trên mặt robot, chính giữa thân) -->
     <link name="imu_link"/>
     <joint name="imu_joint" type="fixed">
         <parent link="base_link"/>
         <child link="imu_link"/>
-        <origin xyz="0.13 0.0 0.27" rpy="0 0 0"/>
+        <origin xyz="0.0 0.0 0.35" rpy="0 0 0"/>
     </joint>
     <!-- End IMU -->

Commit message: feat: add mass 4kg for agv

File: mobile_robot/urdf/new_robot_2.xacro (robot description, xacro)
@@ -36,4 +36,5 @@
 	</material>
 <!--define physical properties for robot-->
+	<xacro:property name="robot_mass" value="4"/>
 	<xacro:property name="body_length" value="0.3"/>
 	<xacro:property name="body_width" value="0.4"/>
@@ -73,4 +74,9 @@
 	<link name="base_link">
        	<origin xyz="0.0 0.0 0.0"/>
+       	<inertial>
+       		<origin xyz="0.0 0.0 0.0" rpy="0.0 0.0 0.0"/>
+       		<mass value="${robot_mass}"/>
+       		<inertia ixx="0.1" ixy="0.0" ixz="0.0" iyy="0.1" iyz="0.0" izz="0.1"/>
+       	</inertial>
     </link>
 <!--chassis link - Frame Structure with Grid-->
